Commit message: add speed limitations

File: car_nav2_mecanum/urdf/mycar.urdf (robot description, URDF)
Before this commit: robot mycar, 10 links, 9 joints
Links:
- link base_link: geometry collision box size=.4 .2 .1; visual mesh filename=model://car/meshes/mycar.dae
- link front_left_wheel: geometry collision sphere radius=.1; visual mesh filename=model://car/meshes/mecanum_wheel_left.STL scale=0.002 .002 0.002
- link front_right_wheel: geometry collision sphere radius=.1; visual mesh filename=model://car/meshes/mecanum_wheel_right.STL scale=0.002 .002 0.002
- link rear_left_wheel: geometry collision sphere radius=.1; visual mesh filename=model://car/meshes/mecanum_wheel_right.STL scale=0.002 .002 0.002
- link rear_right_wheel: geometry collision sphere radius=.1; visual mesh filename=model://car/meshes/mecanum_wheel_left.STL scale=0.002 .002 0.002
- link scan_link: geometry collision box size=.1 .1 .1; visual mesh filename=model://car/meshes/lidar.dae

Commit message: add camera drivers

File: car_nav2_mecanum/urdf/mycar.urdf (robot description, URDF)
Before this commit: robot mycar, 10 links, 9 joints
Links:
- added link ultrasonic_link, mass 0.01; collision box size=0.02 0.05 0.02; visual box size=0.02 0.05 0.02
Joints:
- added joint ultrasonic_joint: type fixed, parent base_link, child ultrasonic_link, origin xyz=0.2 0 0.08 rpy=0 0 0

Commit message: make the new autonomous work with simulation

File: car_nav2_mecanum/urdf/mycar.urdf (robot description, URDF)
Before this commit: robot mycar, 11 links, 10 joints
Joints:
- joint ultrasonic_joint: origin xyz=0.2 0 0.08 rpy=0 0 0 -> xyz=0.2 0 0.001 rpy=0 0 0
